File: Power Board.brd (EAGLE design)
At the start: 100 x 80 mm, 4 parts

Commit message: Initial layout
Parts:
- added C2, C3, C5, C6: 10uF, SparkFun-Capacitors:1206
- added C4: 1uF, SparkFun-Capacitors:1206
- added NEG-GND, NEG-OUT, POS-GND, POS-OUT: BANNANA, PowerSupply:BANNANA
- added R2: (no value), SparkFun-Resistors:1206
- added U$1, U$2: POT, PowerSupply:POT
- added U$10, U$11, U$12, U$9: DIODE-SCHOTTKY, PowerSupply:DIODE-SCHOTTKY
- added U$3: C14_POWER_CONNECTOR, PowerSupply:PANEL_FOR_POWER
- added U$4: TRANSFORMER, PowerSupply:TRANSFORMER
- added U$5, U$6, U$7, U$8: DIODE, PowerSupply:DIODE
- C1: value (none) -> 1uF
Connections:
- new net GND: C1.2, C2.2, C3.2, C4.2, C5.2, C6.2, U$1.P$1, U$2.P$1
- new net N$1: U$3.P$3, U$4.L
- new net N$11: C6.1, LM337.P$4, R2.2, U$10.C, U$12.A
- new net N$12: C5.1, LM337.P$2, R2.1, U$12.C, U$2.P$3
- new net N$2: U$3.P$1, U$4.N
- new net N$3: U$4.+, U$5.A, U$7.C
- new net N$4: C1.1, LM317.P$4, U$5.C, U$8.C, U$9.C
- new net N$5: U$4.-, U$6.C, U$8.A
- new net N$6: C3.1, LM317.P$1, LM317.P$3, R1.2, U$11.C, U$9.A
- new net N$7: C4.1, LM337.P$1, LM337.P$3, U$10.A, U$6.A, U$7.A
- new net N$8: C2.1, LM317.P$2, R1.1, U$1.P$3, U$11.A

Commit message: Updates
Parts:
- added 3.3V_LINEAR_REG: 3.3_LIN_REG, PowerSupply:3.3_LINEAR_REG
- added C10, C7: 2700uF, SparkFun-Capacitors:CPOL-RADIAL-1000UF-63V
- added C11, C12: 2.2uF, SparkFun-Capacitors:1206
- added C13, C14: 10uF, SparkFun-Capacitors:1206
- added C15, C16, C8, C9: .1uF, SparkFun-Capacitors:1206
- added F1, F2: PTCPTH, SparkFun-PowerIC:PTC
- added JP1: FTDI Basic, SparkFun:1X06
- added LED1: (no value), LilyPad-Wearables:LED-1206
- added Q1: 8/16/20MHz, Testing:RESONATOR-SMD-1:1
- added R10, R11, R6, R8: 1M, SparkFun-Resistors:1206
- added R12, R13: 171K, SparkFun-Resistors:1206
- added R14, R15, R16, R3: 10K, SparkFun-Resistors:1206
- added R4, R5: .2, SparkFun-Resistors:1206
- added R7, R9: 220K, SparkFun-Resistors:1206
- added S1, S2, S3: Reset, Testing:TACTILE-SWITCH-SMD-ALT01
- added U$14: SWITCH, PowerSupply:SWITCH
- added U$16: 4-DIGIT_7_SEG, PowerSupply:4-DIGIT_7-SEG
- added U1: ATMEGA328, SparkFun:TQFP32-08
- R1: value (none) -> 227
- U$1, U$2: value POT -> 5k
- moved NEG-GND 203.2 mm to (58.4, 8.89)
- moved U$4 201.4 mm to (85.1, 69.8)
- moved NEG-OUT 198.4 mm to (73.7, 7.62)
- moved POS-GND 180.6 mm to (38.1, 10.2)
- moved POS-OUT 157.3 mm to (24.1, 10.2)
- moved U$2 150.1 mm to (91.4, 5.08)
- moved U$3 149.8 mm to (38.1, 63.5)
- moved LM337 114.3 mm to (91.4, 33.0)
- moved LM317 87.5 mm to (55.9, 50.8)
- moved R1 62.4 mm to (47.0, 41.9)
- moved U$1 55.1 mm to (11.4, 5.08)
Connections:
- removed net N$4: C1.1, LM317.P$4, U$5.C, U$8.C, U$9.C
- new net 3.3V: R12.1, R13.1, R15.2
- new net AREF: C8.2, U1.20
- new net CURR_SENSE_+: C11.2, R6.1, R7.2, U1.23
- new net CURR_SENSE_-: R10.1, R12.2, U1.25
- new net CURR_SENS_-: C6.1, LM337.P$4, R10.2, R2.2, R5.2, U$10.C, U$12.A
- new net CUR_SENS_+: C3.1, LM317.P$1, LM317.P$3, R1.2, R4.2, R6.2, U$11.C, U$9.A
- new net DTR: C15.1, JP1.1
- new net N$10: Q1.3, U1.8
- new net N$13: Q1.1, U1.7
- new net N$14: U$16.P$4, U1.22
- new net N$15: U1.32
- new net N$16: U$16.P$6, U1.1
- new net N$17: U$16.P$7, U1.2
- new net N$18: U$16.P$8, U1.9
- new net N$19: U$16.P$9, U1.10
- new net N$20: U$16.P$10, U1.11
- new net N$21: U$16.P$11, U1.12
- new net N$22: U$16.P$12, U1.13
- new net N$23: U$16.P$13, U1.14
- new net N$24: U$16.P$14, U1.15
- new net N$25: F1.P$2, POS-OUT.P$1, POS-OUT.P$2, POS-OUT.P$3, POS-OUT.P$4
- new net N$26: F2.P$2, NEG-OUT.P$1, NEG-OUT.P$2, NEG-OUT.P$3, NEG-OUT.P$4
- new net N$27: U$14.P$1, U$4.L
- new net N$29: R15.1, S3.3, S3.4, U1.16
- new net N$9: U$16.P$2, U1.28
- new net NEG_IN: C10.2, C4.1, LM337.P$1, LM337.P$3, U$10.A, U$6.A, U$7.A
- new net POS_IN: 3.3V_LINEAR_REG.P$3, C1.1, C13.1, C7.1, LM317.P$4, U$5.C, U$8.C, U$9.C
- new net RESET: C15.2, R3.1, S1.3, S1.4, U1.29
- new net RESET1: R14.1, S2.3, S2.4, U1.17
- new net RXI: JP1.3, U1.30
- new net TXO: JP1.2, U1.31
- new net VCC: 3.3V_LINEAR_REG.P$2, 3.3V_LINEAR_REG.P$4, C14.1, C16.2, C9.2, JP1.4, R14.2, R16.2, R3.2, U1.18, U1.4, U1.6
- new net V_SENSE_+: C12.2, R8.1, R9.2, U1.24
- new net V_SENSE_-: R11.1, R13.2, U1.26
- new net V_SENS_+: F1.P$1, R4.1, R8.2
- new net V_SENS_-: F2.P$1, R11.2, R5.1
- net GND: now also 3.3V_LINEAR_REG.P$1, C10.1, C11.1, C12.1, C13.2, C14.2, C16.1, C7.2, C8.1, C9.1, JP1.5, JP1.6, LED1.C, NEG-GND.P$1, NEG-GND.P$2, NEG-GND.P$3, NEG-GND.P$4, POS-GND.P$1, POS-GND.P$2, POS-GND.P$3, POS-GND.P$4, Q1.2, R9.1, S1.1, S1.2, S2.1, S2.2, S3.1, S3.2, U1.21, U1.3, U1.5
- net N$1: now also U$14.P$2; no longer U$4.L
- net N$11: now also U$16.P$3, U1.19; no longer C6.1, LM337.P$4, R2.2, U$10.C, U$12.A
- net N$6: now also U$16.P$1, U1.27; no longer C3.1, LM317.P$1, LM317.P$3, R1.2, U$11.C, U$9.A
- net N$7: now also LED1.A, R16.1; no longer C4.1, LM337.P$1, LM337.P$3, U$10.A, U$6.A, U$7.A

Commit message: Initial board layout placement
Parts:
- removed U$10, U$11, U$12, U$9: DIODE-SCHOTTKY, PowerSupply:DIODE-SCHOTTKY
- added C17, C18: 2.2uF, SparkFun-Capacitors:1206
- added U$13, U$19, U$20, U$21: DIODE, PowerSupply:DIODE
- R1: value 227 -> 390
- R12, R13: value 171K -> 174K
- R2: value (none) -> 390
- moved C16 386.5 mm to (64.8, 44.5), turned to 90 degrees
- moved R15 354.1 mm to (95.2, 10.2), turned to 180 degrees
- moved C14 350.1 mm to (72.4, 55.9), turned to 180 degrees
- moved R16 350.0 mm to (52.1, 14.0), turned to 180 degrees
- moved C8 349.9 mm to (64.8, 52.1), turned to 90 degrees
- moved LED1 347.0 mm to (59.7, 11.4), turned to 180 degrees
- moved C15 337.6 mm to (44.5, 52.1), turned to 90 degrees
- moved C9 337.6 mm to (44.5, 44.5), turned to 270 degrees
- moved C13 333.5 mm to (72.4, 40.6), turned to 180 degrees
- moved R12 324.1 mm to (88.9, 38.1)
- moved R13 321.0 mm to (88.9, 30.5)
- moved R10 319.3 mm to (96.5, 34.3)
- moved R11 319.3 mm to (96.5, 30.5)
- moved R14 319.1 mm to (24.1, 11.4)
- moved C11 297.0 mm to (38.1, 52.1), turned to 90 degrees
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Connections:
- net 3.3V: now also C17.1, C18.1
- net CURR_SENSE_-: now also C17.2
- net CURR_SENS_-: now also U$20.C, U$21.A; no longer U$10.C, U$12.A
- net CUR_SENS_+: now also U$13.A, U$19.C; no longer U$11.C, U$9.A
- net N$12: now also U$21.C; no longer U$12.C
- net N$8: now also U$19.A; no longer U$11.A
- net NEG_IN: now also U$20.A; no longer U$10.A
- net POS_IN: now also U$13.C; no longer U$9.C
- net V_SENSE_-: now also C18.2
Other:
- board size 100 x 80 mm -> 121.6 x 80 mm

Commit message: Started traces
Connections:
- net GND: now also U$4.GND
Routing:
- net N$27: track 0.00 -> 68.2 mm
- net N$2: track 0.00 -> 67.0 mm
- net POS_IN: track 0.00 -> 51.0 mm
- net N$1: track 0.00 -> 45.9 mm
- net N$5: track 0.00 -> 21.4 mm
- net N$3: track 0.00 -> 19.4 mm
- net NEG_IN: track 0.00 -> 6.35 mm
- added copper zone on layer 1, net N$4
Changed lines of the file:
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@@
 <element name="C6" library="SparkFun-Capacitors" package="1206" value="10uF" x="77.47" y="5.08" rot="R270"/>
 <element name="U$3" library="PowerSupply" package="PANEL_FOR_POWER" value="C14_POWER_CONNECTOR" x="59.69" y="62.23"/>
-<element name="U$4" library="PowerSupply" package="TRANSFORMER" value="TRANSFORMER" x="102.87" y="71.12"/>
 <element name="U$5" library="PowerSupply" package="DIODE" value="DIODE" x="90.17" y="60.96" rot="R90"/>
 <element name="U$6" library="PowerSupply" package="DIODE" value="DIODE" x="102.87" y="60.96" rot="R90"/>
@@
 <element name="C17" library="SparkFun-Capacitors" package="1206" value="2.2uF" x="88.9" y="34.29"/>
 <element name="C18" library="SparkFun-Capacitors" package="1206" value="2.2uF" x="88.9" y="26.67"/>
+<element name="U$4" library="PowerSupply" package="TRANSFORMER" value="TRANSFORMER" x="102.87" y="71.12"/>
 </elements>
 <signals>
 <signal name="N$2">
+<contactref element="U$3" pad="P$1"/>
 <contactref element="U$4" pad="N"/>
-<contactref element="U$3" pad="P$1"/>
-<wire x1="52.69" y1="62.23" x2="102.87" y2="71.12" width="0" layer="19" extent="1-1"/>
+<wire x1="52.69" y1="62.23" x2="56.5" y2="58.42" width="2.54" layer="16"/>
+<wire x1="56.5" y1="58.42" x2="100.17" y2="58.42" width="2.54" layer="16"/>
+<wire x1="100.17" y1="58.42" x2="112.87" y2="71.12" width="2.54" layer="16"/>
 </signal>
 <signal name="N$3">
-<contactref element="U$4" pad="+"/>
 <contactref element="U$5" pad="A"/>
 <contactref element="U$7" pad="C"/>
-<wire x1="96.52" y1="65.46" x2="97.87" y2="76.12" width="0" layer="19" extent="1-1"/>
-<wire x1="90.17" y1="60.96" x2="96.52" y2="65.46" width="0" layer="19" extent="1-1"/>
+<contactref element="U$4" pad="+"/>
+<wire x1="97.87" y1="76.12" x2="97.87" y2="67.39" width="2.54" layer="1"/>
+<wire x1="97.87" y1="67.39" x2="96.52" y2="66.04" width="2.54" layer="1"/>
+<wire x1="96.52" y1="66.04" x2="96.52" y2="65.46" width="2.54" layer="1"/>
+<wire x1="96.52" y1="65.46" x2="95.94" y2="65.46" width="2.54" layer="1"/>
+<wire x1="95.94" y1="65.46" x2="91.44" y2="60.96" width="2.54" layer="1"/>
+<wire x1="91.44" y1="60.96" x2="90.17" y2="60.96" width="2.54" layer="1"/>
 </signal>
 <signal name="POS_IN">
@@
 <contactref element="C13" pad="1"/>
 <contactref element="U$13" pad="C"/>
-<wire x1="90.17" y1="65.46" x2="109.22" y2="65.46" width="0" layer="19" extent="1-1"/>
-<wire x1="96.52" y1="50.8" x2="90.17" y2="65.46" width="0" layer="19" extent="1-1"/>
-<wire x1="78.5" y1="45.77" x2="96.52" y2="50.8" width="0" layer="19" extent="1-1"/>
+<wire x1="90.17" y1="65.46" x2="88.32" y2="65.46" width="2.54" layer="1"/>
+<wire x1="88.32" y1="65.46" x2="85.09" y2="62.23" width="2.54" layer="1"/>
+<wire x1="85.09" y1="62.23" x2="85.09" y2="58.42" width="2.54" layer="1"/>
+<wire x1="85.09" y1="58.42" x2="87.63" y2="55.88" width="2.54" layer="1"/>
+<wire x1="87.63" y1="55.88" x2="111.76" y2="55.88" width="2.54" layer="1"/>
+<wire x1="111.76" y1="55.88" x2="114.3" y2="58.42" width="2.54" layer="1"/>
+<wire x1="114.3" y1="58.42" x2="114.3" y2="60.96" width="2.54" layer="1"/>
+<wire x1="114.3" y1="60.96" x2="110.49" y2="64.77" width="2.54" layer="1"/>
+<wire x1="110.49" y1="64.77" x2="109.91" y2="64.77" width="2.54" layer="1"/>
+<wire x1="109.91" y1="64.77" x2="109.22" y2="65.46" width="2.54" layer="1"/>
+<wire x1="87.63" y1="55.88" x2="96.52" y2="50.8" width="0" layer="19" extent="1-1"/>
+<wire x1="78.5" y1="45.77" x2="87.63" y2="55.88" width="0" layer="19" extent="1-1"/>
 <wire x1="73.79" y1="40.64" x2="78.5" y2="45.77" width="0" layer="19" extent="1-1"/>
 <wire x1="18.92" y1="38.1" x2="73.79" y2="40.64" width="0" layer="19" extent="1-1"/>
@@
 <contactref element="U$8" pad="A"/>
 <contactref element="U$4" pad="-"/>
-<wire x1="102.87" y1="65.46" x2="107.87" y2="76.12" width="0" layer="19" extent="1-1"/>
-<wire x1="109.22" y1="60.96" x2="102.87" y2="65.46" width="0" layer="19" extent="1-1"/>
+<wire x1="109.22" y1="60.96" x2="107.37" y2="60.96" width="2.54" layer="1"/>
+<wire x1="107.37" y1="60.96" x2="102.87" y2="65.46" width="2.54" layer="1"/>
+<wire x1="102.87" y1="65.46" x2="103.56" y2="65.46" width="2.54" layer="1"/>
+<wire x1="103.56" y1="65.46" x2="107.95" y2="69.85" width="2.54" layer="1"/>
+<wire x1="107.95" y1="69.85" x2="107.95" y2="76.04" width="2.54" layer="1"/>
+<wire x1="107.95" y1="76.04" x2="107.87" y2="76.12" width="2.54" layer="1"/>
 </signal>
 <signal name="GND">
@@
 <contactref element="LED1" pad="C"/>
 <contactref element="C16" pad="1"/>
+<contactref element="U$4" pad="GND"/>
+<wire x1="114.3" y1="50.8" x2="102.87" y2="71.12" width="0" layer="19" extent="1-1"/>
 <wire x1="88.9" y1="50.8" x2="114.3" y2="50.8" width="0" layer="19" extent="1-1"/>
 <wire x1="73.9" y1="45.77" x2="88.9" y2="50.8" width="0" layer="19" extent="1-1"/>
@@
 <contactref element="U$3" pad="P$3"/>
 <contactref element="U$14" pad="P$2"/>
-<wire x1="27.29" y1="69.37" x2="66.69" y2="62.23" width="0" layer="19" extent="1-1"/>
+<wire x1="66.69" y1="62.23" x2="55.26" y2="73.66" width="2.54" layer="16"/>
+<wire x1="55.26" y1="73.66" x2="31.58" y2="73.66" width="2.54" layer="16"/>
+<wire x1="31.58" y1="73.66" x2="27.29" y2="69.37" width="2.54" layer="16"/>
 </signal>
 <signal name="N$27">
 <contactref element="U$14" pad="P$1"/>
 <contactref element="U$4" pad="L"/>
-<wire x1="27.29" y1="64.77" x2="92.87" y2="71.12" width="0" layer="19" extent="1-1"/>
+<wire x1="92.87" y1="71.12" x2="87.63" y2="71.12" width="2.54" layer="1"/>
+<wire x1="87.63" y1="71.12" x2="82.55" y2="66.04" width="2.54" layer="1"/>
+<wire x1="82.55" y1="66.04" x2="28.56" y2="66.04" width="2.54" layer="1"/>
+<wire x1="28.56" y1="66.04" x2="27.29" y2="64.77" width="2.54" layer="1"/>
 </signal>
 <signal name="RESET1">
@@
 <contactref element="C10" pad="2"/>
 <contactref element="U$20" pad="A"/>
-<wire x1="96.52" y1="60.96" x2="102.87" y2="60.96" width="0" layer="19" extent="1-1"/>
 <wire x1="106.68" y1="50.8" x2="102.87" y2="60.96" width="0" layer="19" extent="1-1"/>
 <wire x1="106.68" y1="36.83" x2="106.68" y2="50.8" width="0" layer="19" extent="1-1"/>
@@
 <wire x1="99.06" y1="25.4" x2="106.68" y2="26.23" width="0" layer="19" extent="1-1"/>
 <wire x1="106.68" y1="17.65" x2="106.68" y2="26.23" width="0" layer="19" extent="1-1"/>
+<wire x1="96.52" y1="60.96" x2="102.87" y2="60.96" width="2.54" layer="1"/>
 </signal>
 <signal name="N$7">
@@
 <wire x1="53.47" y1="13.97" x2="61.19" y2="11.43" width="0" layer="19" extent="1-1"/>
 </signal>
+<signal name="N$4">
+<polygon width="0.6096" layer="1">
+<vertex x="130.81" y="-19.05"/>
+<vertex x="130.81" y="97.79"/>
+<vertex x="-19.05" y="97.79"/>
+<vertex x="-19.05" y="-2.54"/>
+<vertex x="-19.05" y="-21.59"/>
+<vertex x="130.81" y="-21.59"/>
+</polygon>
+</signal>
 </signals>

Commit message: Finished routing
Parts:
- moved C3 40.2 mm to (8.89, 27.9), turned to 180 degrees
- moved C6 20.5 mm to (95.2, 15.2), turned to 0 degrees
- moved Q1 6.35 mm to (48.3, 40.6), turned to 0 degrees
- moved C13 3.81 mm to (76.2, 40.6)
- moved C14 3.81 mm to (76.2, 55.9)
- moved LED1 1.27 mm to (59.7, 10.2), turned to 0 degrees
- turned C4 to 270 degrees
- turned C8 to 270 degrees
- turned R4 to 180 degrees
- turned R6 to 180 degrees
- turned R8 to 180 degrees
Connections:
- removed net N$16: U$16.P$6, U1.1
- removed net N$17: U$16.P$7, U1.2
- new net N$28: U$16.P$3, U1.1
- new net N$4: U$16.P$14, U1.9
- net N$11: now also U$16.P$6; no longer U$16.P$3
- net N$14: now also U$16.P$7; no longer U$16.P$4
- net N$18: now also U$16.P$10, U1.13; no longer U$16.P$8, U1.9
- net N$19: now also U$16.P$13; no longer U$16.P$9
- net N$20: now also U$16.P$12; no longer U$16.P$10
- net N$22: now also U$16.P$9, U1.14; no longer U$16.P$12, U1.13
- net N$23: now also U$16.P$8, U1.15; no longer U$16.P$13, U1.14
- net N$24: now also U$16.P$4, U1.2; no longer U$16.P$14, U1.15
Routing:
- net GND: track 0.00 -> 729.2 mm, vias 0 -> 33
- net VCC: track 0.00 -> 226.3 mm, vias 0 -> 5
- net POS_IN: track 51.0 -> 197.0 mm, vias 0 -> 5
- net RESET1: track 0.00 -> 91.2 mm, vias 0 -> 4
- net RESET: track 0.00 -> 91.1 mm, vias 0 -> 3
- net N$8: track 0.00 -> 76.7 mm, vias 0 -> 5
- net V_SENSE_-: track 0.00 -> 75.8 mm, vias 0 -> 2
- net N$29: track 0.00 -> 75.5 mm, vias 0 -> 2
- net CUR_SENS_+: track 0.00 -> 75.2 mm
- net CURR_SENS_-: track 0.00 -> 63.9 mm, vias 0 -> 4
- net CURR_SENSE_+: track 0.00 -> 61.2 mm, vias 0 -> 2
- net N$6: track 0.00 -> 57.5 mm, vias 0 -> 2
- net N$9: track 0.00 -> 54.0 mm, vias 0 -> 2
- net NEG_IN: track 6.35 -> 59.2 mm
- net CURR_SENSE_-: track 0.00 -> 49.7 mm, vias 0 -> 2
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- removed copper zone on layer 1, net N$4

Commit message: Some fixes, and Gerbers
Connections:
- net GND: now also R7.1
- net N$15: now also U$16.P$5
Routing:
- net N$15: track 0.00 -> 66.8 mm, vias 0 -> 3
- net N$6: track 57.5 -> 62.0 mm, vias 2 -> 5
- net RESET: track 91.1 -> 93.7 mm
- net DTR: track 43.4 -> 44.9 mm, vias 0 -> 2
- net CUR_SENS_+: track 75.2 -> 76.6 mm
- net RXI: track 49.3 -> 50.1 mm
- net CURR_SENSE_+: track 61.2 -> 62.0 mm
- net V_SENSE_-: track 75.8 -> 76.3 mm
- net V_SENSE_+: track 41.8 -> 42.3 mm, vias 2 -> 4
- net N$8: vias 5 -> 7

Commit message: planes added
Parts:
- JP1: value FTDI Basic -> FTDI
Routing:
- net GND: track 729.4 -> 719.8 mm
- net NEG_IN: track 59.2 -> 60.5 mm
- added copper zone on layer 1, net CUR_SENS_+
- added copper zone on layer 1, net GND
- added copper zone on layer 1, net NEG_IN
Other:
- board text added: "Designed By"
- board text added: "Kyle Rakos"
- board text added: "Power"
- board text added: "Toggle 1"
- board text added: "Toggle 2"
