File: Power Board.brd (EAGLE design)
At the start: 121.6 x 80 mm, 64 parts, among them Q1 8/16/20MHz, U1 ATMEGA328

Commit message: Some part updates and rerouting
Connections:
- net N$1: now also U$14.P$3; no longer U$14.P$2
- net N$27: now also U$14.P$4; no longer U$14.P$1
Routing:
- net N$9: track 54.0 -> 87.9 mm, vias 2 -> 7
- net N$27: track 68.2 -> 74.8 mm, vias 0 -> 1
- net N$1: track 45.9 -> 51.7 mm
- net RESET1: track 91.2 -> 86.3 mm
- net V_SENSE_+: track 42.3 -> 45.3 mm
- net POS_IN: track 197.0 -> 200.0 mm
- net N$28: track 36.9 -> 39.8 mm
- net N$24: track 38.4 -> 35.5 mm
- net N$6: track 62.0 -> 64.5 mm
- net DTR: track 44.9 -> 47.2 mm
- net TXO: vias 1 -> 3
