File: Power Board.sch (EAGLE design)
At the start: 4 parts

Commit message: Initial layout
Parts:
- added C2, C3, C5, C6: 10uF, SparkFun-Capacitors:CAP1206
- added C4: 1uF, SparkFun-Capacitors:CAP1206
- added NEG-GND, NEG-OUT, POS-GND, POS-OUT: BANNANA, PowerSupply:BANNANA
- added R2: (no value), SparkFun-Resistors:RESISTOR1206
- added U$1, U$2: POT, PowerSupply:POT
- added U$10, U$11, U$12, U$9: DIODE-SCHOTTKY, PowerSupply:DIODE-SCHOTTKY
- added U$3: C14_POWER_CONNECTOR, PowerSupply:C14_POWER_CONNECTOR
- added U$4: TRANSFORMER, PowerSupply:TRANSFORMER
- added U$5, U$6, U$7, U$8: DIODE, PowerSupply:DIODE
- C1: value (none) -> 1uF
Connections:
- new net GND: C1.2, C2.2, C3.2, C4.2, C5.2, C6.2, U$1.A, U$2.A
- new net N$1: U$3.LINE, U$4.1
- new net N$11: C6.1, LM337.OUT, R2.2, U$10.C, U$12.A
- new net N$12: C5.1, LM337.ADJ, R2.1, U$12.C, U$2.E
- new net N$2: U$3.NEUTRAL, U$4.2
- new net N$3: U$4.5, U$5.A, U$7.C
- new net N$4: C1.1, LM317.IN, U$5.C, U$8.C, U$9.C
- new net N$5: U$4.3, U$6.C, U$8.A
- new net N$6: C3.1, LM317.OUT, R1.2, U$11.C, U$9.A
- new net N$7: C4.1, LM337.IN, U$10.A, U$6.A, U$7.A
- new net N$8: C2.1, LM317.ADJ, R1.1, U$1.E, U$11.A
Other:
- note added: "TO DO: Add power caps"
- moved on the sheet: C1, LM317, LM337, R1

Commit message: Updates
Parts:
- added 3.3V_LINEAR_REG: 3.3_LIN_REG, PowerSupply:3.3_LIN_REG
- added C10, C7: 2700uF, SparkFun-Capacitors:CAP_POLPTH3
- added C11, C12: 2.2uF, SparkFun-Capacitors:CAP1206
- added C13, C14: 10uF, SparkFun-Capacitors:CAP1206
- added C15, C16, C8, C9: .1uF, SparkFun-Capacitors:CAP1206
- added F1, F2: PTCPTH, SparkFun-PowerIC:PTCPTH
- added JP1: FTDI Basic, SparkFun:ARDUINO_SERIAL_PROGRAMPTH
- added LED1: (no value), LilyPad-Wearables:LED1206
- added Q1: 8/16/20MHz, Testing:RESONATOR1:1
- added R10, R11, R6, R8: 1M, SparkFun-Resistors:RESISTOR1206
- added R12, R13: 171K, SparkFun-Resistors:RESISTOR1206
- added R14, R15, R16, R3: 10K, SparkFun-Resistors:RESISTOR1206
- added R4, R5: .2, SparkFun-Resistors:RESISTOR1206
- added R7, R9: 220K, SparkFun-Resistors:RESISTOR1206
- added S1, S2, S3: Reset, Testing:SWITCH-MOMENTARY-2SMD-ALT01
- added U$14: SWITCH, PowerSupply:SWITCH
- added U$16: 4-DIGIT_7_SEG, PowerSupply:4-DIGIT_7_SEG
- added U1: ATMEGA328, SparkFun:ATMEGA168
- R1: value (none) -> 227
- U$1, U$2: value POT -> 5k
Connections:
- removed net N$4: C1.1, LM317.IN, U$5.C, U$8.C, U$9.C
- new net 3.3V: R12.1, R13.1, R15.2
- new net AREF: C8.2, U1.AREF
- new net CURR_SENSE_+: C11.2, R6.1, R7.2, U1.PC0(ADC0)
- new net CURR_SENSE_-: R10.1, R12.2, U1.PC2(ADC2)
- new net CURR_SENS_-: C6.1, LM337.OUT, R10.2, R2.2, R5.2, U$10.C, U$12.A
- new net CUR_SENS_+: C3.1, LM317.OUT, R1.2, R4.2, R6.2, U$11.C, U$9.A
- new net DTR: C15.1, JP1.DTR
- new net N$10: Q1.3, U1.PB7(XTAL2/TOSC2)
- new net N$13: Q1.1, U1.PB6(XTAL1/TOSC1)
- new net N$14: U$16.C, U1.ADC7
- new net N$15: U1.PD2(INT0)
- new net N$16: U$16.DIG4, U1.PD3(INT1)
- new net N$17: U$16.7_AN, U1.PD4(XCK/T0)
- new net N$18: U$16.8_CAT, U1.PD5(T1)
- new net N$19: U$16.B, U1.PD6(AIN0)
- new net N$20: U$16.DIG3, U1.PD7(AIN1)
- new net N$21: U$16.DIG2, U1.PB0(ICP)
- new net N$22: U$16.F, U1.PB1(OC1A)
- new net N$23: U$16.A, U1.PB2(SS/OC1B)
- new net N$24: U$16.DIG1, U1.PB3(MOSI/OC2)
- new net N$25: F1.2, POS-OUT.P$1
- new net N$26: F2.2, NEG-OUT.P$1
- new net N$27: U$14.O, U$4.1
- new net N$29: R15.1, S3.2, U1.PB4(MISO)
- new net N$9: U$16.D, U1.PC5(ADC5/SCL)
- new net NEG_IN: C10.-, C4.1, LM337.IN, U$10.A, U$6.A, U$7.A
- new net POS_IN: 3.3V_LINEAR_REG.IN, C1.1, C13.1, C7.+, LM317.IN, U$5.C, U$8.C, U$9.C
- new net RESET: C15.2, R3.1, S1.2, U1.PC6(/RESET)
- new net RESET1: R14.1, S2.2, U1.PB5(SCK)
- new net RXI: JP1.TXO, U1.PD0(RXD)
- new net TXO: JP1.RXI, U1.PD1(TXD)
- new net VCC: 3.3V_LINEAR_REG.OUT, C14.1, C16.2, C9.2, JP1.VCC, R14.2, R16.2, R3.2, U1.AVCC, U1.VCC@1, U1.VCC@2
- new net V_SENSE_+: C12.2, R8.1, R9.2, U1.PC1(ADC1)
- new net V_SENSE_-: R11.1, R13.2, U1.PC3(ADC3)
- new net V_SENS_+: F1.1, R4.1, R8.2
- new net V_SENS_-: F2.1, R11.2, R5.1
- net GND: now also 3.3V_LINEAR_REG.ADJ, C10.+, C11.1, C12.1, C13.2, C14.2, C16.1, C7.-, C8.1, C9.1, JP1.CTS, JP1.GND, LED1.C, NEG-GND.P$1, POS-GND.P$1, Q1.2, R9.1, S1.1, S2.1, S3.1, U1.AGND, U1.GND@1, U1.GND@2
- net N$1: now also U$14.P; no longer U$4.1
- net N$11: now also U$16.DP, U1.ADC6; no longer C6.1, LM337.OUT, R2.2, U$10.C, U$12.A
- net N$6: now also U$16.E, U1.PC4(ADC4/SDA); no longer C3.1, LM317.OUT, R1.2, U$11.C, U$9.A
- net N$7: now also LED1.A, R16.1; no longer C4.1, LM337.IN, U$10.A, U$6.A, U$7.A
Other:
- note added: "MICRO"
- note added: "NOT SCHOTTKY"
- note added: "Negative"
- note added: "Positive"
- note removed: "TO DO: Add power caps"
- moved on the sheet: C4, C5, C6, LM337, R2, U$10, U$12, U$2, U$3, U$4, U$5, U$6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

Commit message: Initial board layout placement
Parts:
- removed U$10, U$11, U$12, U$9: DIODE-SCHOTTKY, PowerSupply:DIODE-SCHOTTKY
- added C17, C18: 2.2uF, SparkFun-Capacitors:CAP1206
- added U$13, U$19, U$20, U$21: DIODE, PowerSupply:DIODE
- R1: value 227 -> 390
- R12, R13: value 171K -> 174K
- R2: value (none) -> 390
Connections:
- net 3.3V: now also C17.1, C18.1
- net CURR_SENSE_-: now also C17.2
- net CURR_SENS_-: now also U$20.C, U$21.A; no longer U$10.C, U$12.A
- net CUR_SENS_+: now also U$13.A, U$19.C; no longer U$11.C, U$9.A
- net N$12: now also U$21.C; no longer U$12.C
- net N$8: now also U$19.A; no longer U$11.A
- net NEG_IN: now also U$20.A; no longer U$10.A
- net POS_IN: now also U$13.C; no longer U$9.C
- net V_SENSE_-: now also C18.2
Other:
- note removed: "NOT SCHOTTKY"

Commit message: Started traces
Connections:
- net GND: now also U$4.4
Changed lines of the file:
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@@
 <part name="C6" library="SparkFun-Capacitors" deviceset="CAP" device="1206" value="10uF"/>
 <part name="U$3" library="PowerSupply" deviceset="C14_POWER_CONNECTOR" device=""/>
-<part name="U$4" library="PowerSupply" deviceset="TRANSFORMER" device=""/>
 <part name="GND1" library="SparkFun-Aesthetics" deviceset="GND" device=""/>
 <part name="U$5" library="PowerSupply" deviceset="DIODE" device=""/>
@@
 <part name="C17" library="SparkFun-Capacitors" deviceset="CAP" device="1206" value="2.2uF"/>
 <part name="C18" library="SparkFun-Capacitors" deviceset="CAP" device="1206" value="2.2uF"/>
+<part name="U$4" library="PowerSupply" deviceset="TRANSFORMER" device=""/>
 </parts>
 <sheets>
@@
 <instance part="C6" gate="G$1" x="419.1" y="-86.36"/>
 <instance part="U$3" gate="G$1" x="-22.86" y="50.8"/>
-<instance part="U$4" gate="G$1" x="12.7" y="50.8"/>
 <instance part="GND1" gate="1" x="27.94" y="48.26"/>
 <instance part="U$5" gate="G$1" x="50.8" y="68.58"/>
@@
 <instance part="C17" gate="G$1" x="406.4" y="-35.56"/>
 <instance part="C18" gate="G$1" x="447.04" y="-35.56"/>
+<instance part="U$4" gate="G$1" x="12.7" y="50.8"/>
 </instances>
 <busses>
@@
 <segment>
 <wire x1="-20.32" y1="53.34" x2="-20.32" y2="43.18" width="0.1524" layer="91"/>
-<pinref part="U$4" gate="G$1" pin="2"/>
 <wire x1="-20.32" y1="43.18" x2="7.62" y2="43.18" width="0.1524" layer="91"/>
 <pinref part="U$3" gate="G$1" pin="NEUTRAL"/>
+<pinref part="U$4" gate="G$1" pin="2"/>
 </segment>
 </net>
 <net name="GND" class="0">
-<segment>
-<pinref part="GND1" gate="1" pin="GND"/>
-<wire x1="22.86" y1="50.8" x2="27.94" y2="50.8" width="0.1524" layer="91"/>
-</segment>
 <segment>
 <pinref part="C1" gate="G$1" pin="2"/>
@@
 <wire x1="-137.16" y1="-45.72" x2="-137.16" y2="-48.26" width="0.1524" layer="91"/>
 </segment>
+<segment>
+<pinref part="GND1" gate="1" pin="GND"/>
+<wire x1="22.86" y1="50.8" x2="27.94" y2="50.8" width="0.1524" layer="91"/>
+<pinref part="U$4" gate="G$1" pin="4"/>
+</segment>
 </net>
 <net name="N$3" class="0">
 <segment>
-<pinref part="U$4" gate="G$1" pin="5"/>
 <wire x1="17.78" y1="58.42" x2="17.78" y2="68.58" width="0.1524" layer="91"/>
 <pinref part="U$5" gate="G$1" pin="A"/>
@@
 <wire x1="43.18" y1="55.88" x2="43.18" y2="68.58" width="0.1524" layer="91"/>
 <junction x="43.18" y="68.58"/>
+<pinref part="U$4" gate="G$1" pin="5"/>
 </segment>
 </net>
@@
 <wire x1="53.34" y1="40.64" x2="63.5" y2="40.64" width="0.1524" layer="91"/>
 <wire x1="63.5" y1="40.64" x2="63.5" y2="50.8" width="0.1524" layer="91"/>
-<pinref part="U$4" gate="G$1" pin="3"/>
 <wire x1="17.78" y1="43.18" x2="17.78" y2="35.56" width="0.1524" layer="91"/>
 <wire x1="17.78" y1="35.56" x2="63.5" y2="35.56" width="0.1524" layer="91"/>
 <wire x1="63.5" y1="35.56" x2="63.5" y2="40.64" width="0.1524" layer="91"/>
 <junction x="63.5" y="40.64"/>
+<pinref part="U$4" gate="G$1" pin="3"/>
 </segment>
 </net>
@@
 <pinref part="U$14" gate="G$1" pin="O"/>
 <pinref part="U$4" gate="G$1" pin="1"/>
-<wire x1="2.54" y1="58.42" x2="7.62" y2="58.42" width="0.1524" layer="91"/>
-</segment>
-</net>
+<wire x1="7.62" y1="58.42" x2="2.54" y2="58.42" width="0.1524" layer="91"/>
+</segment>
+</net>

Commit message: Finished routing
Connections:
- removed net N$16: U$16.DIG4, U1.PD3(INT1)
- removed net N$17: U$16.7_AN, U1.PD4(XCK/T0)
- new net N$28: U$16.DP, U1.PD3(INT1)
- new net N$4: U$16.DIG1, U1.PD5(T1)
- net N$11: now also U$16.DIG4; no longer U$16.DP
- net N$14: now also U$16.7_AN; no longer U$16.C
- net N$18: now also U$16.DIG3, U1.PB1(OC1A); no longer U$16.8_CAT, U1.PD5(T1)
- net N$19: now also U$16.A; no longer U$16.B
- net N$20: now also U$16.F; no longer U$16.DIG3
- net N$22: now also U$16.B, U1.PB2(SS/OC1B); no longer U$16.F, U1.PB1(OC1A)
- net N$23: now also U$16.8_CAT, U1.PB3(MOSI/OC2); no longer U$16.A, U1.PB2(SS/OC1B)
- net N$24: now also U$16.C, U1.PD4(XCK/T0); no longer U$16.DIG1, U1.PB3(MOSI/OC2)

Commit message: Some fixes, and Gerbers
Connections:
- net GND: now also R7.1
- net N$15: now also U$16.G
Changed lines of the file:
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@@
 <wire x1="215.9" y1="111.76" x2="215.9" y2="104.14" width="0.1524" layer="91"/>
 <junction x="185.42" y="111.76"/>
-<pinref part="C11" gate="G$1" pin="1"/>
-<wire x1="149.86" y1="104.14" x2="167.64" y2="104.14" width="0.1524" layer="91"/>
 <pinref part="C12" gate="G$1" pin="1"/>
 <wire x1="185.42" y1="104.14" x2="193.04" y2="104.14" width="0.1524" layer="91"/>
 <junction x="185.42" y="104.14"/>
+<pinref part="C11" gate="G$1" pin="1"/>
+<wire x1="149.86" y1="104.14" x2="167.64" y2="104.14" width="0.1524" layer="91"/>
+<pinref part="R7" gate="G$1" pin="1"/>
+<junction x="167.64" y="104.14"/>
 </segment>
 <segment>
@@
 <segment>
 <pinref part="P+4" gate="G$1" pin="3.3V"/>
-<pinref part="C14" gate="G$1" pin="1"/>
-<wire x1="127" y1="119.38" x2="127" y2="124.46" width="0.1524" layer="91"/>
 <pinref part="3.3V_LINEAR_REG" gate="G$1" pin="OUT"/>
 <wire x1="114.3" y1="124.46" x2="127" y2="124.46" width="0.1524" layer="91"/>
 <wire x1="127" y1="124.46" x2="127" y2="132.08" width="0.1524" layer="91"/>
+<pinref part="C14" gate="G$1" pin="1"/>
+<wire x1="127" y1="119.38" x2="127" y2="124.46" width="0.1524" layer="91"/>
+<junction x="127" y="124.46"/>
 </segment>
 <segment>
@@
 <wire x1="-50.8" y1="-93.98" x2="-58.42" y2="-93.98" width="0.1524" layer="91"/>
 <wire x1="-58.42" y1="-93.98" x2="-58.42" y2="-73.66" width="0.1524" layer="91"/>
-</segment>
-</net>
-<net name="N$15" class="0">
-<segment>
-<pinref part="U1" gate="G$1" pin="PD2(INT0)"/>
-<wire x1="-48.26" y1="-83.82" x2="-86.36" y2="-83.82" width="0.1524" layer="91"/>
 </segment>
 </net>
@@
 </segment>
 </net>
+<net name="N$15" class="0">
+<segment>
+<pinref part="U1" gate="G$1" pin="PD2(INT0)"/>
+<pinref part="U$16" gate="G$1" pin="G"/>
+<wire x1="-86.36" y1="-83.82" x2="-50.8" y2="-83.82" width="0.1524" layer="91"/>
+</segment>
+</net>

Commit message: planes added
Parts:
- JP1: value FTDI Basic -> FTDI
Changed lines of the file:
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@@
 <part name="P+1" library="SparkFun" deviceset="3.3V" device="" value="VCC"/>
 <part name="GND15" library="SparkFun" deviceset="GND" device=""/>
-<part name="JP1" library="SparkFun" deviceset="ARDUINO_SERIAL_PROGRAM" device="PTH" value="FTDI Basic"/>
+<part name="JP1" library="SparkFun" deviceset="ARDUINO_SERIAL_PROGRAM" device="PTH" value="FTDI"/>
 <part name="P+4" library="SparkFun" deviceset="3.3V" device="" value="VCC"/>
 <part name="S1" library="Testing" deviceset="SWITCH-MOMENTARY-2" device="SMD-ALT01" value="Reset"/>
